File: Teensy4.1-example.kicad_sch (KiCad schematic)
At the start: 80 parts, among them IC1 MIMXRT1062DVJ6B, J1 Conn_01x11_Male, J2 Conn_01x11_Male, J3 Conn_01x12_Male, J4 Conn_01x11_Male, J5 Conn_01x11_Male, J6 Conn_01x03_Male, J7 Conn_01x03_Male, P2 D26, Q1 Q_PMOS_GDS_DMP3125L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

Commit message: Update MPN for CAP
Parts:
- C19, C20: MPN CC0603KRX7R6BB224 -> CC0603KRNPO9BN100
Changed lines of the file:
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@@
       (effects (font (size 1.27 1.27)) hide)
     )
-    (property "MPN" "CC0603KRX7R6BB224" (id 5) (at 243.205 312.42 0)
+    (property "MPN" "CC0603KRNPO9BN100" (id 5) (at 243.205 312.42 0)
       (effects (font (size 1.27 1.27)) hide)
     )
@@
       (effects (font (size 1.27 1.27)) hide)
     )
-    (property "MPN" "CC0603KRX7R6BB224" (id 5) (at 243.205 304.8 0)
-      (effects (font (size 1.27 1.27)) hide)
-    )
+    (property "MPN" "CC0603KRNPO9BN100" (id 5) (at 243.205 304.8 0)
+      (effects (font (size 1.27 1.27)) hide)
+    )
